Commit message: fix bug on pendulum design

File: ur5_modified_robot.urdf (robot description, URDF)
Before this commit: robot ur5, 13 links, 12 joints
Links:
- link mass_link: mass 0.05 -> 5
Joints:
- joint ee_pendulum_joint: axis 1 0 0 -> 0 1 0; limit lower=-6.28318530718 upper=6.28318530718 effort=150.0 velocity=3.15 -> lower=-20 upper=20 effort=150.0 velocity=3.15; origin xyz=0.0 0.0 0.0 rpy=0.0 0.0 0.0 -> xyz=0.0 0.0 0.0 rpy=0.0 0.0 1.51
